File: esp32-midi-processor/esp32-midi-processor.kicad_sch (KiCad schematic)
At the start: 50 parts, among them J1 Midi IN 1, J10 USB Shield left, J11 Spare, J12 Display, J2 Midi IN 2, J3 Midi OUT 1, J4 Midi OUT 2, J5 ESP32 right, J6 ESP32 left, J7 Input Voltage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

Commit message: add 7805
Parts:
- added U3: LM7805_TO220, Package_TO_SOT_THT:TO-220-3_Vertical, symbol Regulator_Linear:LM7805_TO220
Connections:
- net GND: now also U3.2 (GND)
- net VIN: now also U3.3 (VO); no longer J7.2 (Pin_2)
- new net: J7.2 (Pin_2), U3.1 (VI)
Changed lines of the file:
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@@
 	(wire
 		(pts
+			(xy 85.09 29.21) (xy 85.09 33.02)
+		)
+		(stroke
+			(width 0)
+			(type default)
+		)
+	)
+	(wire
+		(pts
 			(xy 194.31 68.58) (xy 204.47 68.58)
 		)
@@
 	(wire
 		(pts
-			(xy 59.69 21.59) (xy 67.31 21.59)
+			(xy 59.69 21.59) (xy 77.47 21.59)
 		)
 		(stroke
@@
 	(wire
 		(pts
+			(xy 92.71 21.59) (xy 102.87 21.59)
+		)
+		(stroke
+			(width 0)
+			(type default)
+		)
+	)
+	(wire
+		(pts
 			(xy 269.24 86.36) (xy 271.78 86.36)
 		)
@@
 	(global_label "VIN"
 		(shape input)
-		(at 67.31 21.59 0)
+		(at 102.87 21.59 0)
 		(fields_autoplaced yes)
 		(effects
@@
 		)
 		(property "Intersheetrefs" "${INTERSHEET_REFS}"
-			(at 73.3191 21.59 0)
+			(at 108.8791 21.59 0)
 			(effects
 				(font
@@
 	)
 	(symbol
+		(lib_id "power:GND")
+		(at 85.09 33.02 0)
+		(unit 1)
+		(exclude_from_sim no)
+		(in_bom yes)
+		(on_board yes)
+		(dnp no)
+		(fields_autoplaced yes)
+		(property "Reference" "#PWR037"
+			(at 85.09 39.37 0)
+			(effects
+				(font
+					(size 1.27 1.27)
+				)
+				(hide yes)
+			)
+		)
+		(property "Value" "GND"
+			(at 85.09 38.1 0)
+			(effects
+				(font
+					(size 1.27 1.27)
+				)
+			)
+		)
+		(property "Footprint" ""
+			(at 85.09 33.02 0)
+			(effects
+				(font
+					(size 1.27 1.27)
+				)
+				(hide yes)
+			)
+		)
+		(property "Datasheet" ""
+			(at 85.09 33.02 0)
+			(effects
+				(font
+					(size 1.27 1.27)
+				)
+				(hide yes)
+			)
+		)
+		(property "Description" "Power symbol creates a global label with name \"GND\" , ground"
+			(at 85.09 33.02 0)
+			(effects
+				(font
+					(size 1.27 1.27)
+				)
+				(hide yes)
+			)
+		)
+		(pin "1"
+		)
+		(instances
+			(project "esp32-midi-processor"
+				(path "/455de105-8b26-465e-84b2-943a0958c97b"
+					(reference "#PWR037")
+					(unit 1)
+				)
+			)
+		)
+	)
+	(symbol
 		(lib_id "Device:R")
 		(at 46.99 58.42 90)
@@
 					(unit 1)
 				)
+			)
+		)
+	)
+	(symbol
+		(lib_id "Regulator_Linear:LM7805_TO220")
+		(at 85.09 21.59 0)
+		(unit 1)
+		(exclude_from_sim no)
+		(in_bom yes)
+		(on_board yes)
+		(dnp no)
+		(fields_autoplaced yes)
+		(property "Reference" "U3"
+			(at 85.09 15.24 0)
+			(effects
+				(font
+					(size 1.27 1.27)
+				)
+			)
+		)
+		(property "Value" "LM7805_TO220"
+			(at 85.09 17.78 0)
+			(effects
+				(font
+					(size 1.27 1.27)
+				)
+			)
+		)
+		(property "Footprint" "Package_TO_SOT_THT:TO-220-3_Vertical"
+			(at 85.09 15.875 0)
+			(effects
+				(font
+					(size 1.27 1.27)
+					(italic yes)
+				)
+				(hide yes)
+			)
+		)
+		(property "Datasheet" "https://www.onsemi.cn/PowerSolutions/document/MC7800-D.PDF"
+			(at 85.09 22.86 0)
+			(effects
+				(font
+					(size 1.27 1.27)
+				)
+				(hide yes)
+			)
+		)
+		(property "Description" "Positive 1A 35V Linear Regulator, Fixed Output 5V, TO-220"
+			(at 85.09 21.59 0)
+			(effects
+				(font
+					(size 1.27 1.27)
+				)
+				(hide yes)
+			)
+		)
+		(pin "2"
+		)
+		(pin "1"
+		)
+		(pin "3"
+		)
+		(instances
+			(project ""
+				(path "/455de105-8b26-465e-84b2-943a0958c97b"
+					(reference "U3")
+					(unit 1)
+				)

Commit message: add title to schematic
Other:
- title: (none) -> ESP32 Midi Processor
Changed lines of the file:
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@@
 (kicad_sch
-	(version 20231120)
+	(version 20250114)
 	(generator "eeschema")
-	(generator_version "8.0")
+	(generator_version "9.0")
 	(paper "A4")
+	(title_block
+		(title "ESP32 Midi Processor")
+	)
 	(junction
 		(at 137.16 49.53)
@@
 		)
 	)
+	(embedded_fonts no)
 )

Commit message: finish pcb
Parts:
- removed J11: Spare, Connector_PinHeader_2.54mm:PinHeader_1x05_P2.54mm_Vertical, symbol Connector:Conn_01x05_Socket
- added J13: Spare, Connector_PinHeader_2.54mm:PinHeader_1x04_P2.54mm_Vertical, symbol Connector:Conn_01x04_Socket
- U1, U2: footprint Package_DIP:DIP-8_W7.62mm_Socket -> Package_SO:SOP-8_6.605x9.655mm_P2.54mm
Connections:
- net D13 is gone; now on net GPX: J6.13 (Pin_13)
- net +3V3: now also J13.2 (Pin_2)
- net D2: now also J13.4 (Pin_4)
- net D4: now also J13.3 (Pin_3)
- net GND: now also J13.1 (Pin_1)
- net GPX: now reaches J9.3 (Pin_3)
- no-connect marks 27 -> 26
Other:
- note added: "USB Conn"
Changed lines of the file:
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@@
 		(title "ESP32 Midi Processor")
 	)
+	(text "USB Conn"
+		(exclude_from_sim no)
+		(at 176.784 140.97 0)
+		(effects
+			(font
+				(size 1.27 1.27)
+			)
+		)
+	)
+	(text "USB Conn"
+		(exclude_from_sim no)
+		(at 251.46 133.858 0)
+		(effects
+			(font
+				(size 1.27 1.27)
+			)
+		)
+	)
 	(junction
 		(at 137.16 49.53)
@@
 	)
 	(no_connect
-		(at 237.49 142.24)
-	)
-	(no_connect
 		(at 269.24 118.11)
 	)
@@
 	(wire
 		(pts
-			(xy 149.86 166.37) (xy 149.86 171.45)
+			(xy 152.4 166.37) (xy 152.4 173.99)
 		)
 		(stroke
@@
 	(wire
 		(pts
+			(xy 237.49 142.24) (xy 242.57 142.24)
+		)
+		(stroke
+			(width 0)
+			(type default)
+		)
+	)
+	(wire
+		(pts
 			(xy 96.52 111.76) (xy 96.52 118.11)
 		)
@@
 	(wire
 		(pts
-			(xy 154.94 167.64) (xy 154.94 171.45)
-		)
-		(stroke
-			(width 0)
-			(type default)
-		)
-	)
-	(wire
-		(pts
 			(xy 279.4 91.44) (xy 281.94 91.44)
 		)
@@
 	(wire
 		(pts
-			(xy 157.48 162.56) (xy 157.48 171.45)
+			(xy 157.48 162.56) (xy 157.48 173.99)
 		)
 		(stroke
@@
 	(wire
 		(pts
-			(xy 152.4 166.37) (xy 152.4 171.45)
+			(xy 154.94 166.37) (xy 154.94 173.99)
 		)
 		(stroke
@@
 	(wire
 		(pts
-			(xy 160.02 171.45) (xy 160.02 168.91)
+			(xy 160.02 168.91) (xy 160.02 173.99)
 		)
 		(stroke
@@
 		)
 	)
+	(global_label "GPX"
+		(shape input)
+		(at 242.57 142.24 0)
+		(fields_autoplaced yes)
+		(effects
+			(font
+				(size 1.27 1.27)
+			)
+			(justify left)
+		)
+		(property "Intersheetrefs" "${INTERSHEET_REFS}"
+			(at 249.3047 142.24 0)
+			(effects
+				(font
+					(size 1.27 1.27)
+				)
+				(justify left)
+				(hide yes)
+			)
+		)
+	)
 	(global_label "SW2"
 		(shape input)
@@
 		)
 	)
-	(global_label "D13"
+	(global_label "GPX"
 		(shape input)
 		(at 165.1 132.08 180)
@@
 		)
 		(property "Intersheetrefs" "${INTERSHEET_REFS}"
-			(at 158.4258 132.08 0)
+			(at 158.3653 132.08 0)
 			(effects
 				(font
@@
 	(global_label "D2"
 		(shape input)
-		(at 149.86 166.37 90)
+		(at 152.4 166.37 90)
 		(fields_autoplaced yes)
 		(effects
@@
 		)
 		(property "Intersheetrefs" "${INTERSHEET_REFS}"
-			(at 149.86 160.9053 90)
+			(at 152.4 160.9053 90)
 			(effects
 				(font
@@
 		)
 	)
-	(global_label "D13"
-		(shape input)
-		(at 154.94 167.64 90)
-		(fields_autoplaced yes)
-		(effects
-			(font
-				(size 1.27 1.27)
-			)
-			(justify left)
-		)
-		(property "Intersheetrefs" "${INTERSHEET_REFS}"
-			(at 154.94 160.9658 90)
-			(effects
-				(font
-					(size 1.27 1.27)
-				)
-				(justify left)
-				(hide yes)
-			)
-		)
-	)
 	(global_label "D16"
 		(shape input)
@@
 	(global_label "D4"
 		(shape input)
-		(at 152.4 166.37 90)
+		(at 154.94 166.37 90)
 		(fields_autoplaced yes)
 		(effects
@@
 		)
 		(property "Intersheetrefs" "${INTERSHEET_REFS}"
-			(at 152.4 160.9053 90)
+			(at 154.94 160.9053 90)
 			(effects
 				(font
@@
 			)
 		)
-		(property "Footprint" "Package_DIP:DIP-8_W7.62mm_Socket"
+		(property "Footprint" "Package_SO:SOP-8_6.605x9.655mm_P2.54mm"
 			(at 83.566 68.58 0)
 			(effects
@@
 			)
 		)
-		(property "Footprint" "Package_DIP:DIP-8_W7.62mm_Socket"
+		(property "Footprint" "Package_SO:SOP-8_6.605x9.655mm_P2.54mm"
 			(at 84.836 121.92 0)
 			(effects
@@
 	)
 	(symbol
-		(lib_id "Connector:Conn_01x05_Socket")
-		(at 154.94 176.53 270)
+		(lib_id "Switch:SW_Push")
+		(at 151.13 60.96 0)
 		(unit 1)
 		(exclude_from_sim no)
@@
 		(on_board yes)
 		(dnp no)
-		(property "Reference" "J11"
-			(at 146.304 173.99 0)
+		(fields_autoplaced yes)
+		(property "Reference" "SW3"
+			(at 151.13 53.34 0)
 			(effects
 				(font
@@
 			)
 		)
-		(property "Value" "Spare"
-			(at 156.21 178.054 90)
+		(property "Value" "SW_Push"
+			(at 151.13 55.88 0)
 			(effects
 				(font
@@
 			)
 		)
-		(property "Footprint" "Connector_PinHeader_2.54mm:PinHeader_1x05_P2.54mm_Vertical"
-			(at 154.94 176.53 0)
+		(property "Footprint" "Button_Switch_THT:SW_PUSH-12mm_Wuerth-430476085716"
+			(at 151.13 55.88 0)
 			(effects
 				(font
@@
 		)
 		(property "Datasheet" "~"
-			(at 154.94 176.53 0)
+			(at 151.13 55.88 0)
 			(effects
 				(font
@@
 			)
 		)
-		(property "Description" "Generic connector, single row, 01x05, script generated"
-			(at 154.94 176.53 0)
+		(property "Description" "Push button switch, generic, two pins"
+			(at 151.13 60.96 0)
 			(effects
 				(font
@@
 		(pin "1"
 		)
-		(pin "3"
-		)
-		(pin "4"
-		)
-		(pin "5"
-		)
 		(instances
 			(project "esp32-midi-processor"
 				(path "/455de105-8b26-465e-84b2-943a0958c97b"
-					(reference "J11")
+					(reference "SW3")
 					(unit 1)
 				)
@@
 	)
 	(symbol
-		(lib_id "Switch:SW_Push")
-		(at 151.13 60.96 0)
+		(lib_id "power:+5V")
+		(at 255.27 144.78 0)
 		(unit 1)
 		(exclude_from_sim no)
@@
 		(dnp no)
 		(fields_autoplaced yes)
-		(property "Reference" "SW3"
-			(at 151.13 53.34 0)
+		(property "Reference" "#PWR023"
+			(at 255.27 148.59 0)
 			(effects
 				(font
 					(size 1.27 1.27)
 				)
+				(hide yes)
 			)
 		)
-		(property "Value" "SW_Push"
-			(at 151.13 55.88 0)
+		(property "Value" "+5V"
+			(at 255.27 139.7 0)
 			(effects
 				(font
@@
 			)
 		)
-		(property "Footprint" "Button_Switch_THT:SW_PUSH-12mm_Wuerth-430476085716"
-			(at 151.13 55.88 0)
+		(property "Footprint" ""
+			(at 255.27 144.78 0)
 			(effects
 				(font
@@
 			)
 		)
-		(property "Datasheet" "~"
-			(at 151.13 55.88 0)
+		(property "Datasheet" ""
+			(at 255.27 144.78 0)
 			(effects
 				(font
@@
 			)
 		)
-		(property "Description" "Push button switch, generic, two pins"
-			(at 151.13 60.96 0)
+		(property "Description" "Power symbol creates a global label with name \"+5V\""
+			(at 255.27 144.78 0)
 			(effects
 				(font
@@
 			)
 		)
-		(pin "2"
-		)
 		(pin "1"
 		)
@@
 			(project "esp32-midi-processor"
 				(path "/455de105-8b26-465e-84b2-943a0958c97b"
-					(reference "SW3")
+					(reference "#PWR023")
 					(unit 1)
 				)
@@
 	)
 	(symbol
-		(lib_id "power:+5V")
-		(at 255.27 144.78 0)
+		(lib_id "Connector:Conn_01x04_Socket")
+		(at 157.48 179.07 270)
 		(unit 1)
 		(exclude_from_sim no)
@@
 		(dnp no)
 		(fields_autoplaced yes)
-		(property "Reference" "#PWR023"
-			(at 255.27 148.59 0)
+		(property "Reference" "J13"
+			(at 156.21 181.61 90)
 			(effects
 				(font
 					(size 1.27 1.27)
 				)
-				(hide yes)
 			)
 		)
-		(property "Value" "+5V"
-			(at 255.27 139.7 0)
+		(property "Value" "Spare"
+			(at 156.21 184.15 90)
 			(effects
 				(font
@@
 			)
 		)
-		(property "Footprint" ""
-			(at 255.27 144.78 0)
+		(property "Footprint" "Connector_PinHeader_2.54mm:PinHeader_1x04_P2.54mm_Vertical"
+			(at 157.48 179.07 0)
 			(effects
 				(font
@@
 			)
 		)
-		(property "Datasheet" ""
-			(at 255.27 144.78 0)
+		(property "Datasheet" "~"
+			(at 157.48 179.07 0)
 			(effects
 				(font
@@
 			)
 		)
-		(property "Description" "Power symbol creates a global label with name \"+5V\""
-			(at 255.27 144.78 0)
+		(property "Description" "Generic connector, single row, 01x04, script generated"
+			(at 157.48 179.07 0)
 			(effects
 				(font
@@
 			)
 		)
+		(pin "2"
+		)
+		(pin "3"
+		)
+		(pin "4"
+		)
 		(pin "1"
 		)
 		(instances
-			(project "esp32-midi-processor"
+			(project ""
 				(path "/455de105-8b26-465e-84b2-943a0958c97b"
-					(reference "#PWR023")
+					(reference "J13")
 					(unit 1)
 				)
